Commit message: [Fix] Include ur_robot_driver again to solve issue with robot bringup and roslaunch files.

File: src/ur_description/urdf/inc/ur_macro.xacro (robot description, xacro)
@@ -225,5 +225,5 @@
            link/frame) to introduce the necessary rotation over Z (of pi rad).
       -->
-      <origin xyz="0 0 0" rpy="0 0 ${pi}" />
+      <origin xyz="0 0 0" rpy="0 0 ${pi/2.0}" />
     </joint>
     <joint name="${prefix}shoulder_pan_joint" type="revolute">
@@ -344,8 +344,5 @@
       <child link="${prefix}tool0" />
     </joint>
-    <xacro:include filename="$(find ur_description)/urdf/tools.urdf.xacro">
-      <xacro:arg name="prefix" value="${prefix}" />
-      <xacro:arg name="ee_tool" value="${ee_tool}" />
-    </xacro:include>
+    <xacro:include filename="$(find ur_description)/urdf/tools.urdf.xacro" />
   </xacro:macro>
 </robot>

File: src/ur_description/urdf/tools.urdf.xacro (robot description, xacro)
@@ -1,7 +1,7 @@
 <?xml version="1.0"?>
 <robot xmlns:xacro="http://ros.org/wiki/xacro">
+    <xacro:include filename="$(find laser_description)/urdf/ee_laser.urdf.xacro" />
     <xacro:if value="${ee_tool == 'logi_laser'}">
-        <xacro:include filename="$(find laser_description)/urdf/ee_laser.urdf.xacro" />
-        <xacro:ee_laser />
+        <xacro:ee_laser prefix="${prefix}" />
     </xacro:if>
 </robot>

File: src/ur_description/urdf/ur.xacro (robot description, xacro)
@@ -18,7 +18,9 @@
       <xacro:arg name="safety_pos_margin" default="0.15" />
       <xacro:arg name="safety_k_position" default="20" />
+      <xacro:arg name="ee_tool" default="none" />
       <!-- arm -->
       <xacro:ur_robot
             prefix=""
+            ee_tool="$(arg ee_tool)"
             joint_limits_parameters_file="$(arg joint_limit_params)"
             kinematics_parameters_file="$(arg kinematics_params)"

File: src/ur_description/urdf/ur5.xacro (robot description, xacro)
@@ -1,5 +1,4 @@
 <?xml version="1.0"?>
 <robot xmlns:xacro="http://wiki.ros.org/xacro" name="ur5_robot">
-  <xacro:property name="prefix" />
   <xacro:arg name="ee_tool" default="none" />
   <!--

Commit message: [Feat] Add a virtual link inside srdf to act as the end effector and adapt the tools.

File: src/ur_description/urdf/inc/ur_macro.xacro (robot description, xacro)
@@ -344,5 +344,15 @@
       <child link="${prefix}tool0" />
     </joint>
-    <xacro:include filename="$(find ur_description)/urdf/tools.urdf.xacro" />
+    <xacro:if value="${ee_tool != 'none'}">
+      <xacro:include filename="$(find ur_description)/urdf/tools.urdf.xacro" />
+    </xacro:if>
+    <xacro:if value="${ee_tool == 'none'}">
+      <link name="${prefix}virtual_link" />
+      <joint name="${prefix}tool0-virtual_link" type="fixed">
+        <parent link="${prefix}tool0" />
+        <child link="${prefix}virtual_link" />
+        <origin rpy="0 0 0" xyz="0 0 0" />
+      </joint>
+    </xacro:if>
   </xacro:macro>
 </robot>

Commit message: [Feat] Add force-torque sensor to the URDF.

File: src/ur_description/urdf/inc/ur_macro.xacro (robot description, xacro)
@@ -344,4 +344,39 @@
       <child link="${prefix}tool0" />
     </joint>
+    <!-- ROS-Industrial 'sensor' frame: attachment point for force-torque sensors -->
+    <!-- TODO Add the force torque sensor using a parameter -->
+    <link name="${prefix}sensor">
+      <visual>
+        <geometry>
+          <mesh
+            filename="package://ur_description/meshes/ur5/visual/force_torque.stl"
+            scale="1 1 1" />
+        </geometry>
+        <!-- Small offset to avoid any collisions between adjacent -->
+        <origin rpy="0 0 0" xyz="0 0 0" />
+        <material name="LightGrey" />
+      </visual>
+      <inertial>
+        <mass value="0.5" />
+        <inertia ixx="0.1" ixy="-0.000000" ixz="-0.000000" iyy="0.1" iyz="-0.000000"
+          izz="0.1" />
+        <origin rpy="0 0 0" xyz="0.0 0.0 0.0" />
+      </inertial>
+      <collision>
+        <geometry>
+          <mesh
+            filename="package://ur_description/meshes/ur5/collision/force_torque.stl"
+            scale="1 1 1" />
+        </geometry>
+        <!-- Small z offset to avoid any collisions between adjacent -->
+        <origin rpy="0 0 0" xyz="0 0 0" />
+      </collision>
+    </link>
+    <joint name="${prefix}tool0-sensor" type="fixed">
+      <!-- default toolframe: X+ left, Y+ up, Z+ front -->
+      <origin xyz="0 0 0.035" rpy="0 0 0" />
+      <parent link="${prefix}tool0" />
+      <child link="${prefix}sensor" />
+    </joint>
     <xacro:if value="${ee_tool != 'none'}">
       <xacro:include filename="$(find ur_description)/urdf/tools.urdf.xacro" />
@@ -349,6 +384,6 @@
     <xacro:if value="${ee_tool == 'none'}">
       <link name="${prefix}virtual_link" />
-      <joint name="${prefix}tool0-virtual_link" type="fixed">
-        <parent link="${prefix}tool0" />
+      <joint name="${prefix}sensor-virtual_link" type="fixed">
+        <parent link="${prefix}sensor" />
         <child link="${prefix}virtual_link" />
         <origin rpy="0 0 0" xyz="0 0 0" />

Commit message: update position ur5

File: src/ur_description/urdf/inc/ur_macro.xacro (robot description, xacro)
@@ -225,5 +225,6 @@
            link/frame) to introduce the necessary rotation over Z (of pi rad).
       -->
-      <origin xyz="0 0 0" rpy="0 0 ${pi/2.0}" />
+      <!-- <origin xyz="0 0 0" rpy="0 0 ${pi/2.0}" /> -->
+      <origin rpy="0 0 1.57" xyz="0.22 0 0.28"/>
     </joint>
     <joint name="${prefix}shoulder_pan_joint" type="revolute">
