Commit message: [Fix] Small adjustments and solve MoveIt configuration.

File: src/ur_moveit_config/config/gazebo_ur5_robot.urdf (robot description, URDF)
Before this commit: robot ur5_robot, 11 links, 10 joints
Links:
- added link sensor, mass 0.5; collision mesh filename=package://ur_description/meshes/ur5/collision/force_torque.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 scale=1 1 1; visual mesh filename=package://ur_description/meshes/ur5/visual/force_torque.stl scale=1 1 1
- added link virtual_link
Joints:
- added joint sensor-virtual_link: type fixed, parent sensor, child virtual_link, origin xyz=0 0 0 rpy=0 0 0
- added joint tool0-sensor: type fixed, parent tool0, child sensor, origin xyz=0 0 0.035 rpy=0 0 0
- joint base_link-base_link_inertia: origin xyz=0 0 0 rpy=0 0 3.141592653589793 -> xyz=0 0 0 rpy=0 0 1.5707963267948966
